File: hardware/ariel.sch (KiCad schematic (older format))
At the start: 19 parts, among them SW1 SW_Push, U1 WeMos_Battery_Shield, U2 Si7020-A20, U3 WeMos_D1_mini, U4 74HC595

Commit message: Fix circuit for WeMos and shift register
Other:
- note added: "WeMos Battery shield is connected to a LiPo battery."
- note removed: "Battery shield is connected to a LiPo battery."
- moved on the sheet: C1, R1, R2, R3, SW1, U2
Changed lines of the file:
@@
 L Device:R_Small R3
 U 1 1 5C7739E8
-P 1600 3250
-F 0 "R3" H 1450 3250 50  0000 L CNN
-F 1 "470" H 1650 3250 50  0000 L CNN
-F 2 "" H 1600 3250 50  0001 C CNN
-F 3 "~" H 1600 3250 50  0001 C CNN
-	1    1600 3250
+P 3400 3250
+F 0 "R3" H 3250 3250 50  0000 L CNN
+F 1 "470" H 3450 3250 50  0000 L CNN
+F 2 "" H 3400 3250 50  0001 C CNN
+F 3 "~" H 3400 3250 50  0001 C CNN
+	1    3400 3250
 	1    0    0    -1
 $EndComp
@@
 L Device:R_Small R1
 U 1 1 5C773C60
-P 1450 3550
-F 0 "R1" V 1350 3500 50  0000 L CNN
-F 1 "1k" V 1550 3500 50  0000 L CNN
-F 2 "" H 1450 3550 50  0001 C CNN
-F 3 "~" H 1450 3550 50  0001 C CNN
-	1    1450 3550
+P 3250 3550
+F 0 "R1" V 3150 3500 50  0000 L CNN
+F 1 "1k" V 3350 3500 50  0000 L CNN
+F 2 "" H 3250 3550 50  0001 C CNN
+F 3 "~" H 3250 3550 50  0001 C CNN
+	1    3250 3550
 	0    1    1    0
 $EndComp
@@
 L Device:R_Small R2
 U 1 1 5C773D83
-P 1450 3850
-F 0 "R2" V 1350 3850 50  0000 C CNN
-F 1 "10k" V 1550 3850 50  0000 C CNN
-F 2 "" H 1450 3850 50  0001 C CNN
-F 3 "~" H 1450 3850 50  0001 C CNN
-	1    1450 3850
+P 3250 3850
+F 0 "R2" V 3150 3850 50  0000 C CNN
+F 1 "10k" V 3350 3850 50  0000 C CNN
+F 2 "" H 3250 3850 50  0001 C CNN
+F 3 "~" H 3250 3850 50  0001 C CNN
+	1    3250 3850
 	0    1    1    0
 $EndComp
@@
 L Device:C_Small C1
 U 1 1 5C773EE5
-P 1900 3850
-F 0 "C1" V 1800 3800 50  0000 L CNN
-F 1 "10u" V 2000 3800 50  0000 L CNN
-F 2 "" H 1900 3850 50  0001 C CNN
-F 3 "~" H 1900 3850 50  0001 C CNN
-	1    1900 3850
+P 3700 3850
+F 0 "C1" V 3600 3800 50  0000 L CNN
+F 1 "10u" V 3800 3800 50  0000 L CNN
+F 2 "" H 3700 3850 50  0001 C CNN
+F 3 "~" H 3700 3850 50  0001 C CNN
+	1    3700 3850
 	0    1    1    0
 $EndComp
@@
 L Switch:SW_Push SW1
 U 1 1 5C85EE0D
-P 2200 3550
-F 0 "SW1" H 2200 3700 50  0000 C CNN
-F 1 "SW_Push" H 2200 3500 50  0000 C CNN
-F 2 "" H 2200 3750 50  0001 C CNN
-F 3 "" H 2200 3750 50  0001 C CNN
-	1    2200 3550
-	1    0    0    -1
-$EndComp
-Wire Wire Line
-	1550 3550 1650 3550
-Wire Wire Line
-	1550 3850 1650 3850
-Wire Wire Line
-	1650 3550 1650 3850
-Connection ~ 1650 3550
-Wire Wire Line
-	1650 3550 2000 3550
-Connection ~ 1650 3850
-Wire Wire Line
-	1650 3850 1800 3850
+P 4000 3550
+F 0 "SW1" H 4000 3700 50  0000 C CNN
+F 1 "SW_Push" H 4000 3500 50  0000 C CNN
+F 2 "" H 4000 3750 50  0001 C CNN
+F 3 "" H 4000 3750 50  0001 C CNN
+	1    4000 3550
+	1    0    0    -1
+$EndComp
+Wire Wire Line
+	3350 3550 3450 3550
+Wire Wire Line
+	3350 3850 3450 3850
+Wire Wire Line
+	3450 3550 3450 3850
+Connection ~ 3450 3550
+Wire Wire Line
+	3450 3550 3800 3550
+Connection ~ 3450 3850
+Wire Wire Line
+	3450 3850 3600 3850
 $Comp
 L power:GND #PWR03
 U 1 1 5C8607DD
-P 2450 3600
-F 0 "#PWR03" H 2450 3350 50  0001 C CNN
-F 1 "GND" H 2455 3427 50  0000 C CNN
-F 2 "" H 2450 3600 50  0001 C CNN
-F 3 "" H 2450 3600 50  0001 C CNN
-	1    2450 3600
-	1    0    0    -1
-$EndComp
-Wire Wire Line
-	2400 3550 2450 3550
-Wire Wire Line
-	2450 3550 2450 3600
-Wire Wire Line
-	1600 3150 2600 3150
-Wire Wire Line
-	2600 3150 2600 3850
-Wire Wire Line
-	2600 3850 2000 3850
+P 4250 3600
+F 0 "#PWR03" H 4250 3350 50  0001 C CNN
+F 1 "GND" H 4255 3427 50  0000 C CNN
+F 2 "" H 4250 3600 50  0001 C CNN
+F 3 "" H 4250 3600 50  0001 C CNN
+	1    4250 3600
+	1    0    0    -1
+$EndComp
+Wire Wire Line
+	4200 3550 4250 3550
+Wire Wire Line
+	4250 3550 4250 3600
+Wire Wire Line
+	3400 3150 4400 3150
+Wire Wire Line
+	4400 3150 4400 3850
+Wire Wire Line
+	4400 3850 3800 3850
 $Comp
 L power:GND #PWR05
@@
 L Sensor_Humidity:Si7020-A20 U2
 U 1 1 5C86A90D
-P 3750 3900
-F 0 "U2" V 3300 3900 50  0000 C CNN
-F 1 "Si7020-A20" V 4250 3900 50  0000 C CNN
-F 2 "Package_DFN_QFN:DFN-6-1EP_3x3mm_P1mm_EP1.5x2.4mm" H 3750 3500 50  0001 C CNN
-F 3 "https://www.silabs.com/documents/public/data-sheets/Si7020-A20.pdf" H 3550 4200 50  0001 C CNN
-	1    3750 3900
-	0    1    1    0
-$EndComp
-NoConn ~ 3450 4000
+P 1600 3900
+F 0 "U2" V 1150 3900 50  0000 C CNN
+F 1 "Si7020-A20" V 2100 3900 50  0000 C CNN
+F 2 "Package_DFN_QFN:DFN-6-1EP_3x3mm_P1mm_EP1.5x2.4mm" H 1600 3500 50  0001 C CNN
+F 3 "https://www.silabs.com/documents/public/data-sheets/Si7020-A20.pdf" H 1400 4200 50  0001 C CNN
+	1    1600 3900
+	0    1    1    0
+$EndComp
+NoConn ~ 1300 4000
 $Comp
 L Device:R_Small R4
@@
 Text Notes 900  850  0    79   ~ 0
 WeMos Battery Shield
-Text Label 4200 3250 0    50   ~ 0
+Text Label 2050 3250 0    50   ~ 0
 I2C_SCL
-Text Label 4200 3400 0    50   ~ 0
+Text Label 2050 3400 0    50   ~ 0
 I2C_SDA
 $Comp
 L power:GND #PWR04
 U 1 1 5C89C91B
-P 3250 3850
-F 0 "#PWR04" H 3250 3600 50  0001 C CNN
-F 1 "GND" H 3255 3677 50  0000 C CNN
-F 2 "" H 3250 3850 50  0001 C CNN
-F 3 "" H 3250 3850 50  0001 C CNN
-	1    3250 3850
-	1    0    0    -1
-$EndComp
-Wire Wire Line
-	3450 3800 3250 3800
-Wire Wire Line
-	3250 3800 3250 3850
+P 1100 3850
+F 0 "#PWR04" H 1100 3600 50  0001 C CNN
+F 1 "GND" H 1105 3677 50  0000 C CNN
+F 2 "" H 1100 3850 50  0001 C CNN
+F 3 "" H 1100 3850 50  0001 C CNN
+	1    1100 3850
+	1    0    0    -1
+$EndComp
+Wire Wire Line
+	1300 3800 1100 3800
+Wire Wire Line
+	1100 3800 1100 3850
 Text Label 6250 2000 0    50   ~ 0
 3_3V
-Text Label 4200 3900 0    50   ~ 0
+Text Label 2050 3900 0    50   ~ 0
 3_3V
 Text Label 9400 1050 0    50   ~ 0
@@
 Wire Wire Line
 	3500 1350 3650 1350
-Text Label 1200 3150 2    50   ~ 0
+Text Label 3000 3150 2    50   ~ 0
 RST
-Text Label 1200 3350 2    50   ~ 0
+Text Label 3000 3350 2    50   ~ 0
 D0
 Text Label 6250 1700 0    50   ~ 0
 D6
-Text Label 1200 3550 2    50   ~ 0
+Text Label 3000 3550 2    50   ~ 0
 D6
-Text Label 1200 3850 2    50   ~ 0
+Text Label 3000 3850 2    50   ~ 0
 3_3V
 Wire Notes Line
@@
 WeMos D1 Mini v3.0.0
 Wire Wire Line
-	1600 3150 1200 3150
-Connection ~ 1600 3150
-Wire Wire Line
-	1600 3350 1200 3350
-Wire Wire Line
-	1350 3550 1200 3550
-Wire Wire Line
-	1350 3850 1200 3850
-Wire Notes Line
-	900  4700 2900 4700
-Wire Notes Line
-	2900 4700 2900 3000
-Wire Notes Line
-	2900 3000 900  3000
-Wire Notes Line
-	900  3000 900  4700
-Text Notes 900  2950 0    79   ~ 0
+	3400 3150 3000 3150
+Connection ~ 3400 3150
+Wire Wire Line
+	3400 3350 3000 3350
+Wire Wire Line
+	3150 3550 3000 3550
+Wire Wire Line
+	3150 3850 3000 3850
+Wire Notes Line
+	2700 4700 4700 4700
+Wire Notes Line
+	4700 4700 4700 3000
+Wire Notes Line
+	4700 3000 2700 3000
+Wire Notes Line
+	2700 3000 2700 4700
+Text Notes 2700 2950 0    79   ~ 0
 Button circuit
 Wire Wire Line
@@
 Wire Notes Line
 	6900 900  6900 2600
-Connection ~ 9250 2350
 Text Notes 6900 850  0    79   ~ 0
 LED Circuit
 Wire Wire Line
-	4050 3900 4200 3900
-Wire Wire Line
-	3650 3400 3650 3250
-Wire Wire Line
-	3850 3400 4200 3400
-Wire Wire Line
-	3650 3250 4200 3250
-Wire Notes Line
-	3050 3000 3050 4700
-Text Notes 3050 2950 0    79   ~ 0
+	1900 3900 2050 3900
+Wire Wire Line
+	1500 3400 1500 3250
+Wire Wire Line
+	1700 3400 2050 3400
+Wire Wire Line
+	1500 3250 2050 3250
+Wire Notes Line
+	900  3000 900  4700
+Text Notes 900  2950 0    79   ~ 0
 Sensor circuit
-Text Notes 1000 4350 0    50   ~ 0
+Text Notes 2800 4350 0    50   ~ 0
 On button press, ESP8266 will wake up and \ndisplay the humidity values in the LEDs.
 Text Notes 1000 2500 0    50   ~ 0
-Battery shield is connected to a LiPo battery.
+WeMos Battery shield is connected to a LiPo battery.
 Text Notes 4350 2550 0    50   ~ 0
 WeMos remains in deep sleep for 6 hours and wakes \nup to sense the humidity value, display it in the LEDs \nand post the value to the cloud.
@@
 	4200 2600 6600 2600
 Wire Notes Line
-	4600 3000 4600 4700
-Wire Notes Line
-	3050 3000 4600 3000
-Wire Notes Line
-	3050 4700 4600 4700
+	2450 3000 2450 4700
+Wire Notes Line
+	900  3000 2450 3000
+Wire Notes Line
+	900  4700 2450 4700
+Wire Bus Line
+	8350 1050 8350 1550
 Wire Bus Line
 	8150 1050 8150 2400
-Wire Bus Line
-	8350 1050 8350 1550
+Connection ~ 9250 2350
 $EndSCHEMATC
