File: hardware/cactus.sch (KiCad schematic (older format))
At the start: 20 parts, among them SW1 SW_Push, U1 WeMos_Battery_Shield, U2 WeMos_D1_mini, U3 74HC595, U4 Si7021_breakout

Commit message: Add mounting holes, more silkscreen annotations
Parts:
- U1: symbol wemos_mini:WeMos_Battery_Shield -> cactus-rescue:WeMos_Battery_Shield-wemos_mini
- U2: symbol wemos_mini:WeMos_D1_mini -> cactus-rescue:WeMos_D1_mini-wemos_mini
- U4: symbol Si7021_breakout_board:Si7021_breakout -> cactus-rescue:Si7021_breakout-Si7021_breakout_board
Changed lines of the file:
@@
 	900  900  3300 900
 $Comp
-L wemos_mini:WeMos_D1_mini U2
+L cactus-rescue:WeMos_D1_mini-wemos_mini U2
 U 1 1 5C9440E1
 P 4800 1700
@@
 Connection ~ 1800 1300
 $Comp
-L wemos_mini:WeMos_Battery_Shield U1
+L cactus-rescue:WeMos_Battery_Shield-wemos_mini U1
 U 1 1 5C954F32
 P 1800 2000
@@
 	6000 900  6000 3000
 $Comp
-L Si7021_breakout_board:Si7021_breakout U4
+L cactus-rescue:Si7021_breakout-Si7021_breakout_board U4
 U 1 1 5C97D9C5
 P 1800 4100
